Commit message: I think this urdf is fine

File: dokalman_library/src/dokalman/urdf/dokalman_description.urdf (robot description, URDF)
Before this commit: robot dokalman, 3 links, 2 joints
Links:
- added link back_gps; visual mesh filename=package://dokalman/meshes/FrontGPS.STL
- added link front_gps; visual mesh filename=package://dokalman/meshes/BackGPS.STL
- added link left_cam; visual mesh filename=package://dokalman/meshes/FLCam.STL
- added link right_cam; visual mesh filename=package://dokalman/meshes/FRCam.STL
- link front_caster: geometry visual mesh filename=package://dokalman/meshes/Caster.STL
Joints:
- added joint back_gps_joint: type fixed, parent base_link, child back_gps, origin xyz=0.0 0.0 0.465 rpy=0 0 0
- added joint front_gps_joint: type fixed, parent base_link, child front_gps, origin xyz=0.6 0.0 0.465 rpy=0 0 0
- added joint left_cam_joint: type fixed, parent base_link, child left_cam, origin xyz=0.5 -0.16 0.465 rpy=0 0 -1
- added joint right_cam_joint: type fixed, parent base_link, child right_cam, origin xyz=0.5 0.16 0.465 rpy=0 0 1
- joint caster_joint: origin xyz=${caster_xoff} 0.0 ${-(base_height/2)} rpy=0 0 0 -> xyz=${caster_xoff} 0.0 0 rpy=0 0 0

Commit message: checkpoint for sdf generation

File: dokalman_library/src/dokalman/urdf/dokalman_description.urdf (robot description, URDF)
Before this commit: robot dokalman, 7 links, 6 joints
Links:
- added link drivewhl_l_link; visual cylinder length=0.04 radius=0.155
- added link drivewhl_r_link; visual cylinder length=0.04 radius=0.155
Joints:
- added joint drivewhl_l_joint: type continuous, parent base_link, child drivewhl_l_link, origin xyz=-0.0 0.265 -0.0 rpy=0 0 0, axis 0 1 0
- added joint drivewhl_r_joint: type continuous, parent base_link, child drivewhl_r_link, origin xyz=-0.0 -0.265 -0.0 rpy=0 0 0, axis 0 1 0
- joint base_joint: origin xyz=0.0 0.0 ${-(wheel_radius+wheel_zoff)} rpy=0 0 0 -> xyz=0.0 0.0 -0.155 rpy=0 0 0
- joint caster_joint: origin xyz=${caster_xoff} 0.0 0 rpy=0 0 0 -> xyz=0.5 0.0 0 rpy=0 0 0

Commit message: yep

File: dokalman_library/src/dokalman/urdf/dokalman_description.urdf (robot description, URDF)
Before this commit: robot dokalman, 9 links, 8 joints
Links:
- link back_gps: mass None -> 0.1
- link base_link: mass None -> 8
- link drivewhl_l_link: mass None -> 1
- link drivewhl_r_link: mass None -> 1
- link front_caster: mass None -> 0.5
- link front_gps: mass None -> 0.1
- link left_cam: mass None -> 0.2
- link right_cam: mass None -> 0.2

File: dokalman_library/src/dokalman/urdf/dokalman_description.xacro (robot description, xacro)
@@ -13,41 +13,50 @@
 <!-- Robot Base -->
 <link name="base_link">
-<visual>
+  <inertial>
+    <origin xyz="0 0 0" rpy="0 0 0"/>
+    <mass value="8"/>
+    <inertia ixx="0.56" ixy="0" ixz="0" iyy="0.38" iyz="0" izz="0.21"/>
+  </inertial>
+  <visual>
     <origin xyz="0 0 0" rpy="0 0 1.5708"/> <!-- 1.5708 radians = 90 degrees -->
     <geometry>
-    <mesh
-        filename="package://dokalman/meshes/base_link.STL" />
+      <mesh filename="package://dokalman/meshes/base_link.STL"/>
     </geometry>
     <material name="Gray">
-    <color rgba="0.5 0.5 0.5 1.0"/>
+      <color rgba="0.5 0.5 0.5 1.0"/>
     </material>
-</visual>
+  </visual>
 </link>
 <!-- Robot Footprint -->
 <link name="base_footprint"/>
 <joint name="base_joint" type="fixed">
-    <parent link="base_link"/>
-    <child link="base_footprint"/>
-    <origin xyz="0.0 0.0 ${-(wheel_radius+wheel_zoff)}" rpy="0 0 0"/>
+  <parent link="base_link"/>
+  <child link="base_footprint"/>
+  <origin xyz="0.0 0.0 ${-(wheel_radius+wheel_zoff)}" rpy="0 0 0"/>
 </joint>
 <!-- Wheels -->
 <xacro:macro name="wheel" params="prefix x_reflect y_reflect">
-<link name="${prefix}_link">
+  <link name="${prefix}_link">
+    <inertial>
+      <origin xyz="0 0 0" rpy="0 0 0"/>
+      <mass value="1"/>
+      <inertia ixx="0.0008" ixy="0" ixz="0" iyy="0.0008" iyz="0" izz="0.00015"/>
+    </inertial>
     <visual>
-    <origin xyz="0 0 0" rpy="${pi/2} 0 0"/>
-    <geometry>
+      <origin xyz="0 0 0" rpy="${pi/2} 0 0"/>
+      <geometry>
         <cylinder radius="${wheel_radius}" length="${wheel_width}"/>
-    </geometry>
-    <material name="Gray">
+      </geometry>
+      <material name="Gray">
         <color rgba="0.5 0.5 0.5 1.0"/>
-    </material>
+      </material>
     </visual>
-</link>
-<joint name="${prefix}_joint" type="continuous">
+  </link>
+  <joint name="${prefix}_joint" type="continuous">
     <parent link="base_link"/>
     <child link="${prefix}_link"/>
     <origin xyz="${x_reflect*wheel_xoff} ${y_reflect*(base_width/2+wheel_ygap)} ${-wheel_zoff}" rpy="0 0 0"/>
     <axis xyz="0 1 0"/>
-</joint>
+  </joint>
 </xacro:macro>
 <xacro:wheel prefix="drivewhl_l" x_reflect="-1" y_reflect="1" />
@@ -55,89 +64,109 @@
 <!-- Caster Wheel -->
 <link name="front_caster">
-<visual>
+  <inertial>
+    <origin xyz="0 0 0" rpy="0 0 0"/>
+    <mass value="0.5"/>
+    <inertia ixx="0.0001" ixy="0" ixz="0" iyy="0.0001" iyz="0" izz="0.0002"/>
+  </inertial>
+  <visual>
     <origin xyz="-0.05 0 -0.16" rpy="1.5708 0 1.5708"/> <!-- 1.5708 radians = 90 degrees -->
     <geometry>
-    <mesh
-        filename="package://dokalman/meshes/Caster.STL" />
+      <mesh filename="package://dokalman/meshes/Caster.STL"/>
     </geometry>
     <material name="Gray">
-    <color rgba="0 1.0 1.0 1.0"/>
+      <color rgba="0 1.0 1.0 1.0"/>
     </material>
-</visual>
+  </visual>
 </link>
 <joint name="caster_joint" type="fixed">
-    <parent link="base_link"/>
-    <child link="front_caster"/>
-    <origin xyz="${caster_xoff} 0.0 0" rpy="0 0 0"/>
+  <parent link="base_link"/>
+  <child link="front_caster"/>
+  <origin xyz="${caster_xoff} 0.0 0" rpy="0 0 0"/>
 </joint>
 <!-- GPS -->
 <link name="back_gps">
-<visual>
+  <inertial>
+    <origin xyz="0 0 0" rpy="0 0 0"/>
+    <mass value="0.1"/>
+    <inertia ixx="0.000001" ixy="0" ixz="0" iyy="0.000001" iyz="0" izz="0.000002"/>
+  </inertial>
+  <visual>
     <origin xyz="-0.025 0.025 0" rpy="1.5708 0 1.5708"/> <!-- 1.5708 radians = 90 degrees -->
     <geometry>
-    <mesh
-        filename="package://dokalman/meshes/FrontGPS.STL" />
+      <mesh filename="package://dokalman/meshes/FrontGPS.STL"/>
     </geometry>
     <material name="Gray">
-    <color rgba="0 1.0 1.0 1.0"/>
+      <color rgba="0 1.0 1.0 1.0"/>
     </material>
-</visual>
+  </visual>
 </link>
 <joint name="back_gps_joint" type="fixed">
-    <parent link="base_link"/>
-    <child link="back_gps"/>
-    <origin xyz="0.0 0.0 0.465" rpy="0 0 0"/>
+  <parent link="base_link"/>
+  <child link="back_gps"/>
+  <origin xyz="0.0 0.0 0.465" rpy="0 0 0"/>
 </joint>
 <link name="front_gps">
-<visual>
+  <inertial>
+    <origin xyz="0 0 0" rpy="0 0 0"/>
+    <mass value="0.1"/>
+    <inertia ixx="0.000001" ixy="0" ixz="0" iyy="0.000001" iyz="0" izz="0.000002"/>
+  </inertial>
+  <visual>
     <origin xyz="0.025 -0.025 0" rpy="1.5708 0 -1.5708"/> <!-- 1.5708 radians = 90 degrees -->
     <geometry>
-    <mesh
-        filename="package://dokalman/meshes/BackGPS.STL" />
+      <mesh filename="package://dokalman/meshes/BackGPS.STL"/>
     </geometry>
     <material name="Gray">
-    <color rgba="0 1.0 1.0 1.0"/>
+      <color rgba="0 1.0 1.0 1.0"/>
     </material>
-</visual>
+  </visual>
 </link>
 <joint name="front_gps_joint" type="fixed">
-    <parent link="base_link"/>
-    <child link="front_gps"/>
-    <origin xyz="0.6 0.0 0.465" rpy="0 0 0"/>
+  <parent link="base_link"/>
+  <child link="front_gps"/>
+  <origin xyz="0.6 0.0 0.465" rpy="0 0 0"/>
 </joint>
 <!-- CAMERAS -->
 <link name="left_cam">
-<visual>
+  <inertial>
+    <origin xyz="0 0 0" rpy="0 0 0"/>
+    <mass value="0.2"/>
+    <inertia ixx="0.000005" ixy="0" ixz="0" iyy="0.000005" iyz="0" izz="0.00001"/>
+  </inertial>
+  <visual>
     <origin xyz="0.01 0.02 0.025" rpy="1.5708 0 1.5708"/> <!-- 1.5708 radians = 90 degrees -->
     <geometry>
-    <mesh
-        filename="package://dokalman/meshes/FLCam.STL" />
+      <mesh filename="package://dokalman/meshes/FLCam.STL"/>
     </geometry>
     <material name="Gray">
-    <color rgba="0 1.0 1.0 1.0"/>
+      <color rgba="0 1.0 1.0 1.0"/>
     </material>
-</visual>
+  </visual>
 </link>
 <joint name="left_cam_joint" type="fixed">
-    <parent link="base_link"/>
-    <child link="left_cam"/>
-    <origin xyz="0.5 -0.16 0.465" rpy="0 0 -1"/>
+  <parent link="base_link"/>
+  <child link="left_cam"/>
+  <origin xyz="0.5 -0.16 0.465" rpy="0 0 -1"/>
 </joint>
 <link name="right_cam">
-<visual>
+  <inertial>
+    <origin xyz="0 0 0" rpy="0 0 0"/>
+    <mass value="0.2"/>
+    <inertia ixx="0.000005" ixy="0" ixz="0" iyy="0.000005" iyz="0" izz="0.00001"/>
+  </inertial>
+  <visual>
     <origin xyz="0.01 0.02 0.025" rpy="1.5708 0 1.5708"/> <!-- 1.5708 radians = 90 degrees -->
     <geometry>
-    <mesh
-        filename="package://dokalman/meshes/FRCam.STL" />
+      <mesh filename="package://dokalman/meshes/FRCam.STL"/>
     </geometry>
     <material name="Gray">
-    <color rgba="0 1.0 1.0 1.0"/>
+      <color rgba="0 1.0 1.0 1.0"/>
     </material>
-</visual>
+  </visual>
 </link>
 <joint name="right_cam_joint" type="fixed">
-    <parent link="base_link"/>
-    <child link="right_cam"/>
-    <origin xyz="0.5 0.16 0.465" rpy="0 0 1"/>
+  <parent link="base_link"/>
+  <child link="right_cam"/>
+  <origin xyz="0.5 0.16 0.465" rpy="0 0 1"/>
 </joint>
 </robot>
