Commit message: urdf loads into gazebo

File: dokalman_library/description/robot_core.xacro (robot description, xacro)
@@ -14,19 +14,21 @@
     <link name="chassis">
         <visual>
-            <origin xyz="0.15 0 0.075"/>
-            <geometry>
-                <box size="0.3 0.3 0.15"/>
-            </geometry>
-            <material name="white"/>
+        <geometry>
+            <mesh filename="file://$(find dokalman_library)/meshes/3DBenchy.stl" scale="0.01 0.01 0.01" />
+        </geometry>
+        <material name="red"/>
         </visual>
         <collision>
-            <origin xyz="0.15 0 0.075"/>
-            <geometry>
-                <box size="0.3 0.3 0.15"/>
-            </geometry>
+        <origin rpy="0 1.5708 0" xyz="0.25 0 0" />
+        <geometry>
+            <cylinder length="0.5" radius="0.05" />
+        </geometry>
+        <material name="red"/>
         </collision>
-        <xacro:inertial_box mass="0.5" x="0.3" y="0.3" z="0.15">
-            <origin xyz="0.15 0 0.075" rpy="0 0 0"/>
-        </xacro:inertial_box>
+        <inertial>
+        <origin xyz="0 0 .25" rpy="0 0 0" />
+        <mass value="1" />
+        <inertia ixx="1.0" ixy="0.0" ixz="0.0" iyy="1.0" iyz="0.0" izz="1.0" />
+        </inertial>
     </link>
     <gazebo reference="chassis">

File: dokalman_library/urdf/DokalmanURDF.urdf.xacro (robot description, xacro)
@@ -4,11 +4,20 @@
      For more information, please see http://wiki.ros.org/sw_urdf_exporter -->
 <robot
-  name="robot">
-  <link
-    name="base_link">
+  name="DokalmanURDF">
+  <link name="base_link">
+  </link>
+  <joint name="chassis_joint" type="fixed">
+    <parent link="base_link"/>
+    <child link="ChassisLink"/>
+    <origin xyz="1.0198E-15 0.007743 0" rpy="0 0 0"/>
+  </joint>
+  <link
+    name="ChassisLink">
     <inertial>
       <origin
         xyz="1.0198E-15 0.007743 0.042916"
         rpy="0 0 0" />
+      <parent
+        link="base_link" />
       <mass
         value="3.8804" />
@@ -27,19 +36,19 @@
       <geometry>
         <mesh
-          filename="package://dokalman_library/meshes/base_link.STL" />
-      </geometry>
-      <material
-        name="">
-        <color
-          rgba="0.79216 0.81961 0.93333 1" />
-      </material>
-    </visual>
-    <collision>
-      <origin
-        xyz="0 0 0"
-        rpy="0 0 0" />
-      <geometry>
-        <mesh
-          filename="package://dokalman_library/meshes/base_link.STL" />
+          filename="file://$(find dokalman_library)/meshes/base_link.STL" />
+      </geometry>
+      <material
+        name="">
+        <color
+          rgba="0.79216 0.81961 0.93333 1" />
+      </material>
+    </visual>
+    <collision>
+      <origin
+        xyz="0 0 0"
+        rpy="0 0 0" />
+      <geometry>
+        <mesh
+          filename="file://$(find dokalman_library)/meshes/base_link.STL" />
       </geometry>
     </collision>
@@ -67,19 +76,19 @@
       <geometry>
         <mesh
-          filename="package://dokalman_library/meshes/BackLeftWheelLink.STL" />
-      </geometry>
-      <material
-        name="">
-        <color
-          rgba="0.79216 0.81961 0.93333 1" />
-      </material>
-    </visual>
-    <collision>
-      <origin
-        xyz="0 0 0"
-        rpy="0 0 0" />
-      <geometry>
-        <mesh
-          filename="package://dokalman_library/meshes/BackLeftWheelLink.STL" />
+          filename="file://$(find dokalman_library)/meshes/BackLeftWheelLink.STL" />
+      </geometry>
+      <material
+        name="">
+        <color
+          rgba="0.79216 0.81961 0.93333 1" />
+      </material>
+    </visual>
+    <collision>
+      <origin
+        xyz="0 0 0"
+        rpy="0 0 0" />
+      <geometry>
+        <mesh
+          filename="file://$(find dokalman_library)/meshes/BackLeftWheelLink.STL" />
       </geometry>
     </collision>
@@ -87,5 +96,5 @@
   <joint
     name="BackLeftWheelJoint"
-    type="revolute">
+    type="continuous">
     <origin
       xyz="-0.2427 -0.30175 -0.26683"
@@ -125,19 +134,19 @@
       <geometry>
         <mesh
-          filename="package://dokalman_library/meshes/BackRightWheelLink.STL" />
-      </geometry>
-      <material
-        name="">
-        <color
-          rgba="0.79216 0.81961 0.93333 1" />
-      </material>
-    </visual>
-    <collision>
-      <origin
-        xyz="0 0 0"
-        rpy="0 0 0" />
-      <geometry>
-        <mesh
-          filename="package://dokalman_library/meshes/BackRightWheelLink.STL" />
+          filename="file://$(find dokalman_library)/meshes/BackRightWheelLink.STL" />
+      </geometry>
+      <material
+        name="">
+        <color
+          rgba="0.79216 0.81961 0.93333 1" />
+      </material>
+    </visual>
+    <collision>
+      <origin
+        xyz="0 0 0"
+        rpy="0 0 0" />
+      <geometry>
+        <mesh
+          filename="file://$(find dokalman_library)/meshes/BackRightWheelLink.STL" />
       </geometry>
     </collision>
@@ -145,5 +154,5 @@
   <joint
     name="BackRightWheelJoint"
-    type="revolute">
+    type="continuous">
     <origin
       xyz="0.2427 -0.30175 -0.26683"
@@ -183,19 +192,19 @@
       <geometry>
         <mesh
-          filename="package://dokalman_library/meshes/CasterLink.STL" />
-      </geometry>
-      <material
-        name="">
-        <color
-          rgba="0.79216 0.81961 0.93333 1" />
-      </material>
-    </visual>
-    <collision>
-      <origin
-        xyz="0 0 0"
-        rpy="0 0 0" />
-      <geometry>
-        <mesh
-          filename="package://dokalman_library/meshes/CasterLink.STL" />
+          filename="file://$(find dokalman_library)/meshes/CasterLink.STL" />
+      </geometry>
+      <material
+        name="">
+        <color
+          rgba="0.79216 0.81961 0.93333 1" />
+      </material>
+    </visual>
+    <collision>
+      <origin
+        xyz="0 0 0"
+        rpy="0 0 0" />
+      <geometry>
+        <mesh
+          filename="file://$(find dokalman_library)/meshes/CasterLink.STL" />
       </geometry>
     </collision>
@@ -203,10 +212,10 @@
   <joint
     name="CasterJoint"
-    type="revolute">
+    type="continuous">
     <origin
       xyz="0 0.3302 -0.21908"
       rpy="1.5708 0 -0.01511" />
     <parent
-      link="base_link" />
+      link="ChassisLink" />
     <child
       link="CasterLink" />
@@ -241,19 +250,19 @@
       <geometry>
         <mesh
-          filename="package://dokalman_library/meshes/FrontLeftWheelLink.STL" />
-      </geometry>
-      <material
-        name="">
-        <color
-          rgba="0.79216 0.81961 0.93333 1" />
-      </material>
-    </visual>
-    <collision>
-      <origin
-        xyz="0 0 0"
-        rpy="0 0 0" />
-      <geometry>
-        <mesh
-          filename="package://dokalman_library/meshes/FrontLeftWheelLink.STL" />
+          filename="file://$(find dokalman_library)/meshes/FrontLeftWheelLink.STL" />
+      </geometry>
+      <material
+        name="">
+        <color
+          rgba="0.79216 0.81961 0.93333 1" />
+      </material>
+    </visual>
+    <collision>
+      <origin
+        xyz="0 0 0"
+        rpy="0 0 0" />
+      <geometry>
+        <mesh
+          filename="file://$(find dokalman_library)/meshes/FrontLeftWheelLink.STL" />
       </geometry>
     </collision>
@@ -261,5 +270,5 @@
   <joint
     name="FrontLeftWheelJoint"
-    type="revolute">
+    type="continuous">
     <origin
       xyz="-0.083806 -0.10265 0.10795"
@@ -299,19 +308,19 @@
       <geometry>
         <mesh
-          filename="package://dokalman_library/meshes/FrontRightWheelLink.STL" />
-      </geometry>
-      <material
-        name="">
-        <color
-          rgba="0.79216 0.81961 0.93333 1" />
-      </material>
-    </visual>
-    <collision>
-      <origin
-        xyz="0 0 0"
-        rpy="0 0 0" />
-      <geometry>
-        <mesh
-          filename="package://dokalman_library/meshes/FrontRightWheelLink.STL" />
+          filename="file://$(find dokalman_library)/meshes/FrontRightWheelLink.STL" />
+      </geometry>
+      <material
+        name="">
+        <color
+          rgba="0.79216 0.81961 0.93333 1" />
+      </material>
+    </visual>
+    <collision>
+      <origin
+        xyz="0 0 0"
+        rpy="0 0 0" />
+      <geometry>
+        <mesh
+          filename="file://$(find dokalman_library)/meshes/FrontRightWheelLink.STL" />
       </geometry>
     </collision>
@@ -319,5 +328,5 @@
   <joint
     name="FrontRightWheelJoint"
-    type="revolute">
+    type="continuous">
     <origin
       xyz="0.083901 -0.10265 0.10795"
