Commit message: cool this kinda works >:(

File: dokalman_library/urdf/DokalmanURDF.urdf.xacro (robot description, xacro)
@@ -217,5 +217,5 @@
       rpy="1.5708 0 -0.01511" />
     <parent
-      link="ChassisLink" />
+      link="base_link" />
     <child
       link="CasterLink" />
@@ -223,6 +223,6 @@
       xyz="0 1 0" />
     <limit
-      lower="-1.57"
-      upper="1.57"
+      lower="0"
+      upper="3.1415"
       effort="1"
       velocity="1" />

File: dokalman_library/urdf/lidar.xacro (robot description, xacro)
@@ -1,51 +1,60 @@
 <?xml version="1.0"?>
 <robot xmlns:xacro="http://www.ros.org/wiki/xacro">
-  <!-- LiDAR Sensor -->
   <link name="lidar_link">
+    <inertial>
+      <origin xyz="0 0 0" rpy="0 0 0"/>
+      <mass value="0.125"/>
+      <inertia ixx="0.001"  ixy="0"  ixz="0" iyy="0.001" iyz="0" izz="0.001" />
+    </inertial>
+    <collision>
+      <origin xyz="0 0 0" rpy="0 0 0"/>
+      <geometry>
+        <cylinder radius="0.0508" length="0.055"/>
+      </geometry>
+    </collision>
     <visual>
+      <origin xyz="0 0 0" rpy="0 0 0"/>
       <geometry>
-        <cylinder length="0.1" radius="0.05"/>
+        <cylinder radius="0.0508" length="0.055"/>
       </geometry>
     </visual>
-    <collision>
-      <geometry>
-        <cylinder length="0.1" radius="0.05"/>
-      </geometry>
-    </collision>
   </link>
-  <!-- Joint to connect LiDAR to the robot -->
   <joint name="lidar_joint" type="fixed">
     <parent link="base_link"/>
     <child link="lidar_link"/>
-    <origin xyz="0 0 0.35" rpy="0 0 0"/> <!-- Adjust position/orientation as needed -->
+    <origin xyz="0 0 0.3" rpy="0 0 0"/>
   </joint>
-  <!-- Gazebo Plugin for LiDAR -->
   <gazebo reference="lidar_link">
-    <sensor type="ray" name="lidar_sensor">
-      <pose>0 0 0 0 0 0</pose>
+    <sensor name="lidar" type="ray">
+      <always_on>true</always_on>
       <visualize>true</visualize>
-      <update_rate>20</update_rate>
+      <update_rate>5</update_rate>
       <ray>
         <scan>
           <horizontal>
-            <samples>720</samples>
-            <resolution>1</resolution>
-            <min_angle>0</min_angle>
-            <max_angle>6.2832</max_angle>
+            <samples>360</samples>
+            <resolution>1.000000</resolution>
+            <min_angle>0.000000</min_angle>
+            <max_angle>6.280000</max_angle>
           </horizontal>
         </scan>
         <range>
-          <min>0.2</min>
-          <max>10.0</max>
-          <resolution>0.01</resolution>
+          <min>0.120000</min>
+          <max>3.5</max>
+          <resolution>0.015000</resolution>
         </range>
+        <noise>
+          <type>gaussian</type>
+          <mean>0.0</mean>
+          <stddev>0.01</stddev>
+        </noise>
       </ray>
-      <plugin name="laser_controller" filename="libgazebo_ros_ray_sensor.so">
-                <ros>
-                    <argument>~/out:=scan</argument>
-                </ros>
-                <output_type>sensor_msgs/LaserScan</output_type>
-                <frame_name>laser_frame</frame_name>
-            </plugin>
+      <plugin name="scan" filename="libgazebo_ros_ray_sensor.so">
+        <ros>
+          <remapping>~/out:=scan</remapping>
+        </ros>
+        <output_type>sensor_msgs/LaserScan</output_type>
+        <frame_name>lidar_link</frame_name>
+      </plugin>
     </sensor>
   </gazebo>
