Commit message: updated some camera config

File: dokalman_library/urdf/DokalmanExtras.xacro (robot description, xacro)
@@ -61,63 +61,3 @@
         <origin xyz="0 -0.35 0.215" rpy="0 0 0"/> <!-- RPY in radians, adjust position and orientation as needed -->
     </joint>
-    <!-- FLCam Link and Joint -->
-    <link name="FLCam">
-        <inertial>
-            <origin xyz="-0.021 0 0.024" rpy="1.5708 0 -3.1415"/>
-            <mass value="0.1"/> <!-- adjust mass as needed -->
-            <inertia ixx="0.0001" ixy="0" ixz="0" iyy="0.0001" iyz="0" izz="0.0001"/> <!-- adjust inertia as needed -->
-        </inertial>
-        <visual>
-            <origin xyz="-0.021 0 0.024" rpy="1.5708 0 -3.1415"/> <!-- RPY in radians -->
-            <geometry>
-            <mesh filename="file://$(find dokalman_library)/meshes/FLCam.STL"/>
-            </geometry>
-            <material
-                name="">
-                <color
-                rgba="0.79216 0.81961 0.93333 1" />
-      </material>
-        </visual>
-        <collision>
-            <origin xyz="-0.021 0 0.024" rpy="1.5708 0 -3.1415"/> <!-- RPY in radians -->
-            <geometry>
-            <mesh filename="file://$(find dokalman_library)/meshes/FLCam.STL"/>
-            </geometry>
-        </collision>
-    </link>
-    <joint name="FLCam_joint" type="fixed">
-        <parent link="base_link"/>
-        <child link="FLCam"/>
-        <origin xyz="-0.18 0.2 0.215" rpy="0 0 1.2"/> <!-- RPY in radians, adjust position and orientation as needed -->
-    </joint>
-    <!-- FRCam Link and Joint -->
-    <link name="FRCam">
-        <inertial>
-            <origin xyz="-0.021 0 0.024" rpy="1.5708 0 -3.1415"/>
-            <mass value="0.1"/> <!-- adjust mass as needed -->
-            <inertia ixx="0.0001" ixy="0" ixz="0" iyy="0.0001" iyz="0" izz="0.0001"/> <!-- adjust inertia as needed -->
-        </inertial>
-        <visual>
-            <origin xyz="-0.021 0 0.024" rpy="1.5708 0 -3.1415"/> <!-- RPY in radians -->
-            <geometry>
-            <mesh filename="file://$(find dokalman_library)/meshes/FRCam.STL"/>
-            </geometry>
-            <material
-                name="">
-                <color
-                rgba="0.79216 0.81961 0.93333 1" />
-      </material>
-        </visual>
-        <collision>
-            <origin xyz="-0.021 0 0.024" rpy="1.5708 0 -3.1415"/> <!-- RPY in radians -->
-            <geometry>
-            <mesh filename="file://$(find dokalman_library)/meshes/FRCam.STL"/>
-            </geometry>
-        </collision>
-    </link>
-    <joint name="FRCam_joint" type="fixed">
-        <parent link="base_link"/>
-        <child link="FRCam"/>
-        <origin xyz="0.18 0.2 0.215" rpy="0 0 -1.2"/> <!-- RPY in radians, adjust position and orientation as needed -->
-    </joint>
 </robot>

File: dokalman_library/urdf/camera.xacro (robot description, xacro)
@@ -6,5 +6,5 @@
         <parent link="ChassisLink"/>
         <child link="left_camera_link"/>
-        <origin xyz="0.23 0.21 0.24" rpy="0 0.3 0.4"/>
+        <origin xyz="0.33 0.00 0.24" rpy="0 ${50*pi/180} ${-pi/2 + pi/2}"/>
     </joint>
     <link name="left_camera_link">
@@ -29,9 +29,9 @@
             <update_rate>10</update_rate>
             <camera>
-                <horizontal_fov>1.089</horizontal_fov>
+                <horizontal_fov>2.094</horizontal_fov>
                 <image>
                     <format>R8G8B8</format>
-                    <width>640</width>
-                    <height>480</height>
+                    <width>1920</width>
+                    <height>1080</height>
                 </image>
                 <clip>
@@ -50,5 +50,5 @@
         <parent link="ChassisLink"/>
         <child link="right_camera_link"/>
-        <origin xyz="-0.23 0.21 0.24" rpy="0 0.3 2.7"/>
+        <origin xyz="-0.33 0.00 0.24" rpy="0 ${50*pi/180} ${pi/2 + pi/2}"/>
     </joint>
     <link name="right_camera_link">
@@ -73,9 +73,9 @@
             <update_rate>10</update_rate>
             <camera>
-                <horizontal_fov>1.089</horizontal_fov>
+                <horizontal_fov>2.094</horizontal_fov>
                 <image>
                     <format>R8G8B8</format>
-                    <width>640</width>
-                    <height>480</height>
+                    <width>1920</width>
+                    <height>1080</height>
                 </image>
                 <clip>
@@ -90,9 +90,9 @@
         </sensor>
     </gazebo>
-<!--Front Camera Stuff-->
+    <!--Front Camera Stuff-->
     <joint name="front_camera_joint" type="fixed">
         <parent link="ChassisLink"/>
         <child link="front_camera_link"/>
-        <origin xyz="0 0.48 0.24" rpy="0 0.3 1.6"/>
+        <origin xyz="0 0.48 0.24" rpy="0 ${50*pi/180} ${0 + pi/2}"/>
     </joint>
     <link name="front_camera_link">
@@ -117,9 +117,9 @@
             <update_rate>10</update_rate>
             <camera>
-                <horizontal_fov>1.089</horizontal_fov>
+                <horizontal_fov>2.094</horizontal_fov>
                 <image>
                     <format>R8G8B8</format>
-                    <width>640</width>
-                    <height>480</height>
+                    <width>1920</width>
+                    <height>1080</height>
                 </image>
                 <clip>

File: dokalman_library/urdf/lidar.xacro (robot description, xacro)
@@ -28,5 +28,5 @@
     <sensor name="lidar" type="ray">
       <always_on>true</always_on>
-      <visualize>true</visualize>
+      <visualize>false</visualize>
       <update_rate>5</update_rate>
       <ray>

Commit message: added base footprint

File: dokalman_library/urdf/DokalmanExtras.xacro (robot description, xacro)
@@ -61,3 +61,10 @@
         <origin xyz="0 -0.35 0.215" rpy="0 0 0"/> <!-- RPY in radians, adjust position and orientation as needed -->
     </joint>
+    <!-- base_footprint Link and Joint -->
+    <link name="base_footprint" />
+    <joint name="base_to_base_footprint" type="fixed">
+        <parent link="base_link"/>
+        <child link="base_footprint"/>
+        <origin xyz="0 0 0" rpy="0 0 0"/> <!-- RPY in radians, adjust position and orientation as needed -->
+    </joint>
 </robot>
