Commit message: fixed lidar joint on dokalman library

File: dokalman_library/urdf/lidar.xacro (robot description, xacro)
@@ -23,6 +23,7 @@
     <parent link="base_link"/>
     <child link="lidar_link"/>
-    <origin xyz="0 0 0.3" rpy="0 0 0"/>
+    <origin xyz="0 0 0.3" rpy="0 0 1.578"/>
   </joint>
+<!--
   <gazebo reference="lidar_link">
     <sensor name="lidar" type="ray">
@@ -58,4 +59,4 @@
       </plugin>
     </sensor>
-  </gazebo>
+  </gazebo> -->
 </robot>
