Commit message: added front camera

File: dokalman_library/urdf/camera.xacro (robot description, xacro)
@@ -90,3 +90,47 @@
         </sensor>
     </gazebo>
+<!--Front Camera Stuff-->
+    <joint name="front_camera_joint" type="fixed">
+        <parent link="ChassisLink"/>
+        <child link="front_camera_link"/>
+        <origin xyz="0 0.48 0.24" rpy="0 0.3 1.6"/>
+    </joint>
+    <link name="front_camera_link">
+        <visual>
+            <geometry>
+                <box size="0.010 0.03 0.03"/>
+            </geometry>
+            <material name="red"/>
+        </visual>
+    </link>
+    <joint name="front_camera_optical_joint" type="fixed">
+        <parent link="front_camera_link"/>
+        <child link="front_camera_link_optical"/>
+        <origin xyz="0 0 0" rpy="${-pi/2} 0 ${-pi/2}"/>
+    </joint>
+    <link name="front_camera_link_optical"></link>
+    <gazebo reference="front_camera_link">
+        <material>Gazebo/Red</material>
+        <sensor name="front_camera" type="camera">
+            <pose> 0 0 0 0 0 0 </pose>
+            <visualize>true</visualize>
+            <update_rate>10</update_rate>
+            <camera>
+                <horizontal_fov>1.089</horizontal_fov>
+                <image>
+                    <format>R8G8B8</format>
+                    <width>640</width>
+                    <height>480</height>
+                </image>
+                <clip>
+                    <near>0.05</near>
+                    <far>8.0</far>
+                </clip>
+            </camera>
+            <plugin name="front_camera_controller" filename="libgazebo_ros_camera.so">
+                <frame_name>front_camera_link_optical</frame_name>
+                <cameraName>front_camera</cameraName>
+            </plugin>
+        </sensor>
+    </gazebo>
 </robot>

Commit message: update camera stuff

File: dokalman_library/urdf/camera.xacro (robot description, xacro)
@@ -2,9 +2,53 @@
 <robot xmlns:xacro="http://www.ros.org/wiki/xacro" >
     <xacro:include filename="materials.xacro"/>
+    <!--Right Camera Stuff-->
+    <joint name="right_camera_joint" type="fixed">
+        <parent link="ChassisLink"/>
+        <child link="right_camera_link"/>
+        <origin xyz="0.33 0.00 0.24" rpy="0 ${50*pi/180} ${-pi/2 + pi/2}"/>
+    </joint>
+    <link name="right_camera_link">
+        <visual>
+            <geometry>
+                <box size="0.010 0.03 0.03"/>
+            </geometry>
+            <material name="red"/>
+        </visual>
+    </link>
+    <joint name="right_camera_optical_joint" type="fixed">
+        <parent link="right_camera_link"/>
+        <child link="right_camera_link_optical"/>
+        <origin xyz="0 0 0" rpy="${-pi/2} 0 ${-pi/2}"/>
+    </joint>
+    <link name="right_camera_link_optical"></link>
+    <gazebo reference="right_camera_link">
+        <material>Gazebo/Red</material>
+        <sensor name="right_camera" type="camera">
+            <pose> 0 0 0 0 0 0 </pose>
+            <visualize>true</visualize>
+            <update_rate>10</update_rate>
+            <camera>
+                <horizontal_fov>2.094</horizontal_fov>
+                <image>
+                    <format>R8G8B8</format>
+                    <width>1920</width>
+                    <height>1080</height>
+                </image>
+                <clip>
+                    <near>0.05</near>
+                    <far>8.0</far>
+                </clip>
+            </camera>
+            <plugin name="right_camera_controller" filename="libgazebo_ros_camera.so">
+                <frame_name>right_camera_link_optical</frame_name>
+                <cameraName>right_camera</cameraName>
+            </plugin>
+        </sensor>
+    </gazebo>
     <!--Left Camera Stuff-->
     <joint name="left_camera_joint" type="fixed">
         <parent link="ChassisLink"/>
         <child link="left_camera_link"/>
-        <origin xyz="0.33 0.00 0.24" rpy="0 ${50*pi/180} ${-pi/2 + pi/2}"/>
+        <origin xyz="-0.33 0.00 0.24" rpy="0 ${50*pi/180} ${pi/2 + pi/2}"/>
     </joint>
     <link name="left_camera_link">
@@ -43,48 +87,4 @@
                 <frame_name>left_camera_link_optical</frame_name>
                 <cameraName>left_camera</cameraName>
-            </plugin>
-        </sensor>
-    </gazebo>
-    <!--Right Camera Stuff-->
-    <joint name="right_camera_joint" type="fixed">
-        <parent link="ChassisLink"/>
-        <child link="right_camera_link"/>
-        <origin xyz="-0.33 0.00 0.24" rpy="0 ${50*pi/180} ${pi/2 + pi/2}"/>
-    </joint>
-    <link name="right_camera_link">
-        <visual>
-            <geometry>
-                <box size="0.010 0.03 0.03"/>
-            </geometry>
-            <material name="red"/>
-        </visual>
-    </link>
-    <joint name="right_camera_optical_joint" type="fixed">
-        <parent link="right_camera_link"/>
-        <child link="right_camera_link_optical"/>
-        <origin xyz="0 0 0" rpy="${-pi/2} 0 ${-pi/2}"/>
-    </joint>
-    <link name="right_camera_link_optical"></link>
-    <gazebo reference="right_camera_link">
-        <material>Gazebo/Red</material>
-        <sensor name="right_camera" type="camera">
-            <pose> 0 0 0 0 0 0 </pose>
-            <visualize>true</visualize>
-            <update_rate>10</update_rate>
-            <camera>
-                <horizontal_fov>2.094</horizontal_fov>
-                <image>
-                    <format>R8G8B8</format>
-                    <width>1920</width>
-                    <height>1080</height>
-                </image>
-                <clip>
-                    <near>0.05</near>
-                    <far>8.0</far>
-                </clip>
-            </camera>
-            <plugin name="right_camera_controller" filename="libgazebo_ros_camera.so">
-                <frame_name>right_camera_link_optical</frame_name>
-                <cameraName>right_camera</cameraName>
             </plugin>
         </sensor>

Commit message: added removing orange cone in image

File: dokalman_library/urdf/camera.xacro (robot description, xacro)
@@ -6,5 +6,5 @@
         <parent link="ChassisLink"/>
         <child link="right_camera_link"/>
-        <origin xyz="0.33 0.00 0.24" rpy="0 ${50*pi/180} ${-pi/2 + pi/2}"/>
+        <origin xyz="0.33 0.00 0.24" rpy="0 ${50*pi/180} ${-64*pi/180 + pi/2}"/>
     </joint>
     <link name="right_camera_link">
@@ -50,5 +50,5 @@
         <parent link="ChassisLink"/>
         <child link="left_camera_link"/>
-        <origin xyz="-0.33 0.00 0.24" rpy="0 ${50*pi/180} ${pi/2 + pi/2}"/>
+        <origin xyz="-0.33 0.00 0.24" rpy="0 ${50*pi/180} ${64*pi/180+ pi/2}"/>
     </joint>
     <link name="left_camera_link">

Commit message: update nuking orange barrel

File: dokalman_library/urdf/camera.xacro (robot description, xacro)
@@ -6,5 +6,5 @@
         <parent link="ChassisLink"/>
         <child link="right_camera_link"/>
-        <origin xyz="0.33 0.00 0.24" rpy="0 ${50*pi/180} ${-64*pi/180 + pi/2}"/>
+        <origin xyz="0.33 0.00 0.24" rpy="0 ${45*pi/180} ${-64*pi/180 + pi/2}"/>
     </joint>
     <link name="right_camera_link">
@@ -50,5 +50,5 @@
         <parent link="ChassisLink"/>
         <child link="left_camera_link"/>
-        <origin xyz="-0.33 0.00 0.24" rpy="0 ${50*pi/180} ${64*pi/180+ pi/2}"/>
+        <origin xyz="-0.33 0.00 0.24" rpy="0 ${45*pi/180} ${64*pi/180+ pi/2}"/>
     </joint>
     <link name="left_camera_link">
@@ -94,5 +94,5 @@
         <parent link="ChassisLink"/>
         <child link="front_camera_link"/>
-        <origin xyz="0 0.48 0.24" rpy="0 ${50*pi/180} ${0 + pi/2}"/>
+        <origin xyz="0 0.48 0.24" rpy="0 ${45*pi/180} ${0 + pi/2}"/>
     </joint>
     <link name="front_camera_link">
