Commit message: added robot footprint to dokalman and some change documentation

File: dokalman_library/src/dokalman_library/urdf/DokalmanURDF.urdf.xacro (robot description, xacro)
@@ -3,7 +3,21 @@
      Commit Version: 1.6.0-4-g7f85cfe  Build Version: 1.6.7995.38578
      For more information, please see http://wiki.ros.org/sw_urdf_exporter -->
+<!--
+  This URDF was also edited by though. This is not the original state of the file.
+  Edits made:
+    - updated joints to be contiunuous
+    - added base footprint joint and link
+    - fixed reference to mesh files paths
+-->
 <robot
   name="DokalmanURDF">
   <link name="base_link">
+  </link>
+  <joint name="base_footprint_joint" type="fixed">
+    <parent link="base_link"/>
+    <child link="base_footprint"/>
+    <origin xyz="0 0 0" rpy="0 0 0"/>
+  </joint>
+  <link name="base_footprint">
   </link>
   <joint name="chassis_joint" type="fixed">
