Commit message: removed the original robot core

File: robot_library/src/articubot_one/description/robot.urdf.xacro (robot description, xacro)
@@ -3,5 +3,5 @@
     <xacro:arg name="use_ros2_control" default="true"/>
     <xacro:arg name="sim_mode" default="false"/>
-    <xacro:include filename="robot_core.xacro" />
+    <!-- <xacro:include filename="robot_core.xacro" /> -->
     <xacro:include filename="dokalman_core.xacro" />
     <xacro:if value="$(arg use_ros2_control)">

File: robot_library/src/articubot_one/description/robot_core.xacro (robot description, xacro)
@@ -2,4 +2,5 @@
 <robot xmlns:xacro="http://www.ros.org/wiki/xacro" >
     <xacro:include filename="inertial_macros.xacro"/>
+<!--
     <xacro:property name="chassis_length" value="0.335"/>
     <xacro:property name="chassis_width" value="0.265"/>
@@ -30,9 +31,9 @@
     <material name="red">
         <color rgba="1 0 0 1"/>
-    </material>
-    <!-- BASE LINK -->
+    </material> -->
+    <!-- BASE LINK
     <link name="base_link">
-    </link>
-    <!-- BASE_FOOTPRINT LINK -->
+    </link>-->
+    <!-- BASE_FOOTPRINT LINK
     <joint name="base_footprint_joint" type="fixed">
         <parent link="base_link"/>
@@ -41,5 +42,5 @@
     </joint>
     <link name="base_footprint">
-    </link>
+    </link>-->
     <!-- CHASSIS LINK
     <joint name="chassis_joint" type="fixed">
