Commit message: wheel changes stage 1

File: robot_library/src/articubot_one/description/dokalman_core.xacro (robot description, xacro)
@@ -2,9 +2,12 @@
 <robot xmlns:xacro="http://www.ros.org/wiki/xacro">
   <xacro:include filename="inertial_macros.xacro"/>
-  <xacro:property name="wheel_radius" value="0.19"/>
-  <xacro:property name="wheel_thickness" value="0.026"/>
-  <xacro:property name="wheel_offset_x" value="0.2427"/>
-  <xacro:property name="wheel_offset_y" value="0.10265"/>
-  <xacro:property name="wheel_offset_z" value="0.10795"/>
+  <!-- PROPERTIES -->
+  <xacro:property name="wheel_radius" value="0.15"/>
+  <xacro:property name="wheel_thickness" value="0.032"/>
+  <xacro:property name="wheel_mass" value="0.15"/>
+  <xacro:property name="wheel_offset_x" value="0.30175"/>
+  <xacro:property name="wheel_offset_y" value="0.2427"/>
+  <xacro:property name="wheel_offset_z" value="0.26683"/>
+  <!-- MATERIALS -->
   <material name="white">
       <color rgba="1 1 1 1" />
@@ -22,4 +25,13 @@
       <color rgba="1 0 0 1"/>
   </material>
+  <!-- BASE LINK -->
+  <link name="base_link"/>
+  <!-- BASE_FOOTPRINT LINK -->
+  <joint name="base_footprint_joint" type="fixed">
+      <parent link="base_link"/>
+      <child link="base_footprint"/>
+      <origin xyz="0 0 0" rpy="0 0 0"/>
+  </joint>
+  <link name="base_footprint"/>
   <!-- CHASSIS -->
   <joint name="dokalman_chassis_joint" type="fixed">
@@ -70,115 +82,55 @@
   </link>
   <!-- BACK LEFT WHEEL -->
-  <link name="BackLeftWheelLink">
-    <inertial>
-      <origin
-        xyz="-0.020955 0 0"
-        rpy="0 0 0" />
-      <mass
-        value="2.9916" />
-      <inertia
-        ixx="0.035119"
-        ixy="0"
-        ixz="0"
-        iyy="0.017802"
-        iyz="0"
-        izz="0.018192" />
-    </inertial>
-    <visual>
-      <origin
-        xyz="0 0 0"
-        rpy="0 0 0" />
-      <geometry>
-        <mesh
-          filename="file://$(find articubot_one)/meshes/BackLeftWheelLink.STL" />
-      </geometry>
-      <material
-        name="">
-        <color
-          rgba="0.79216 0.81961 0.93333 1" />
-      </material>
-    </visual>
-    <collision>
-      <origin
-        xyz="0 0 0"
-        rpy="0 0 0" />
-      <geometry>
-        <mesh
-          filename="file://$(find articubot_one)/meshes/BackLeftWheelLink.STL" />
-      </geometry>
-    </collision>
-  </link>
   <joint name="left_wheel_joint" type="continuous">
-    <origin
-      xyz="-0.30175 0.2427 -0.26683"
-      rpy="0 0 -1.5708" />
-    <parent
-      link="base_link" />
-    <child
-      link="BackLeftWheelLink" />
-    <axis
-      xyz="-1 0 0" />
-    <limit
-      lower="0"
-      upper="3.1415"
-      effort="1"
-      velocity="1" />
-  </joint>
+      <parent link="base_link"/>
+      <child link="left_wheel"/>
+      <origin xyz="0 ${wheel_offset_y} 0" rpy="-${pi/2} 0 0" />
+      <axis xyz="0 0 1"/>
+  </joint>
+  <link name="left_wheel">
+      <visual>
+          <geometry>
+              <cylinder radius="${wheel_radius}" length="${wheel_thickness}"/>
+          </geometry>
+          <material name="blue"/>
+      </visual>
+      <collision>
+          <geometry>
+              <sphere radius="${wheel_radius}"/>
+          </geometry>
+      </collision>
+      <xacro:inertial_cylinder mass="${wheel_mass}" length="${wheel_thickness}" radius="${wheel_radius}">
+          <origin xyz="0 0 0" rpy="0 0 0"/>
+      </xacro:inertial_cylinder>
+  </link>
+  <gazebo reference="left_wheel">
+      <material>Gazebo/Blue</material>
+  </gazebo>
   <!-- BACK RIGHT WHEEL -->
-  <link name="BackRightWheelLink">
-    <inertial>
-      <origin
-        xyz="0.020955 0 0"
-        rpy="0 0 0" />
-      <mass
-        value="2.9916" />
-      <inertia
-        ixx="0.035119"
-        ixy="0"
-        ixz="0"
-        iyy="0.017802"
-        iyz="0"
-        izz="0.018192" />
-    </inertial>
-    <visual>
-      <origin
-        xyz="0 0 0"
-        rpy="0 0 0" />
-      <geometry>
-        <mesh
-          filename="file://$(find articubot_one)/meshes/BackRightWheelLink.STL" />
-      </geometry>
-      <material
-        name="">
-        <color
-          rgba="0.79216 0.81961 0.93333 1" />
-      </material>
-    </visual>
-    <collision>
-      <origin
-        xyz="0 0 0"
-        rpy="0 0 0" />
-      <geometry>
-        <mesh
-          filename="file://$(find articubot_one)/meshes/BackRightWheelLink.STL" />
-      </geometry>
-    </collision>
-  </link>
   <joint name="right_wheel_joint" type="continuous">
-    <origin
-      xyz="-0.30175 -0.2427 -0.26683"
-      rpy="0 0 -1.5708" />
-    <parent
-      link="base_link" />
-    <child
-      link="BackRightWheelLink" />
-    <axis
-      xyz="-1 0 0" />
-    <limit
-      lower="0"
-      upper="3.1415"
-      effort="1"
-      velocity="1" />
-  </joint>
+        <parent link="base_link"/>
+        <child link="right_wheel"/>
+        <origin xyz="0 ${-wheel_offset_y} 0" rpy="${pi/2} 0 0" />
+        <axis xyz="0 0 -1"/>
+    </joint>
+    <link name="right_wheel">
+        <visual>
+            <geometry>
+                <cylinder radius="${wheel_radius}" length="${wheel_thickness}"/>
+            </geometry>
+            <material name="blue"/>
+        </visual>
+        <collision>
+            <geometry>
+                <sphere radius="${wheel_radius}"/>
+            </geometry>
+        </collision>
+        <xacro:inertial_cylinder mass="${wheel_mass}" length="${wheel_thickness}" radius="${wheel_radius}">
+            <origin xyz="0 0 0" rpy="0 0 0"/>
+        </xacro:inertial_cylinder>
+    </link>
+    <gazebo reference="right_wheel">
+        <material>Gazebo/Blue</material>
+    </gazebo>
   <!-- CASTER -->
   <link name="CasterLink">

Commit message: made wheels and diff drive consistent to simulation

File: robot_library/src/articubot_one/description/dokalman_core.xacro (robot description, xacro)
@@ -4,9 +4,9 @@
   <!-- PROPERTIES -->
   <xacro:property name="wheel_radius" value="0.15"/>
-  <xacro:property name="wheel_thickness" value="0.032"/>
+  <xacro:property name="wheel_thickness" value="0.035"/>
   <xacro:property name="wheel_mass" value="0.15"/>
-  <xacro:property name="wheel_offset_x" value="0.30175"/>
-  <xacro:property name="wheel_offset_y" value="0.2427"/>
-  <xacro:property name="wheel_offset_z" value="0.26683"/>
+  <xacro:property name="wheel_offset_x" value="-0.30175"/>
+  <xacro:property name="wheel_offset_y" value="0.26"/>
+  <xacro:property name="wheel_offset_z" value="-0.26683"/>
   <!-- MATERIALS -->
   <material name="white">
@@ -85,5 +85,5 @@
       <parent link="base_link"/>
       <child link="left_wheel"/>
-      <origin xyz="0 ${wheel_offset_y} 0" rpy="-${pi/2} 0 0" />
+      <origin xyz="${wheel_offset_x} ${wheel_offset_y} ${wheel_offset_z}" rpy="-${pi/2} 0 0" />
       <axis xyz="0 0 1"/>
   </joint>
@@ -105,5 +105,5 @@
   </link>
   <gazebo reference="left_wheel">
-      <material>Gazebo/Blue</material>
+      <material>Gazebo/White</material>
   </gazebo>
   <!-- BACK RIGHT WHEEL -->
@@ -111,5 +111,5 @@
         <parent link="base_link"/>
         <child link="right_wheel"/>
-        <origin xyz="0 ${-wheel_offset_y} 0" rpy="${pi/2} 0 0" />
+        <origin xyz="${wheel_offset_x}   ${-wheel_offset_y} ${wheel_offset_z}" rpy="${pi/2} 0 0" />
         <axis xyz="0 0 -1"/>
     </joint>
@@ -131,5 +131,5 @@
     </link>
     <gazebo reference="right_wheel">
-        <material>Gazebo/Blue</material>
+        <material>Gazebo/White</material>
     </gazebo>
   <!-- CASTER -->

File: robot_library/src/articubot_one/description/gazebo_control.xacro (robot description, xacro)
@@ -6,6 +6,6 @@
             <left_joint>left_wheel_joint</left_joint>
             <right_joint>right_wheel_joint</right_joint>
-            <wheel_separation>0.4854</wheel_separation>
-            <wheel_diameter>0.19</wheel_diameter>
+            <wheel_separation>0.52</wheel_separation>
+            <wheel_diameter>0.15</wheel_diameter>
             <!-- Limits -->
             <max_wheel_torque>10</max_wheel_torque>

Commit message: fixed robot's footprint

File: robot_library/src/articubot_one/description/dokalman_core.xacro (robot description, xacro)
@@ -31,5 +31,5 @@
       <parent link="base_link"/>
       <child link="base_footprint"/>
-      <origin xyz="0 0 0" rpy="0 0 0"/>
+      <origin xyz="0 0 -0.40" rpy="0 0 0"/>
   </joint>
   <link name="base_footprint"/>

Commit message: latest changes

File: robot_library/src/articubot_one/description/dokalman_core.xacro (robot description, xacro)
@@ -41,20 +41,7 @@
   </joint>
   <link name="ChassisLink">
-    <inertial>
-      <origin
-        xyz="0 0 0.042916"
-        rpy="0 0 -1.5708" />
-      <parent
-        link="base_link" />
-      <mass
-        value="3.8804" />
-      <inertia
-        ixx="0.46922"
-        ixy="0"
-        ixz="0"
-        iyy="0.43543"
-        iyz="-0.0081395"
-        izz="0.28753" />
-    </inertial>
+    <xacro:inertial_box mass="1.5" x="1.2192" y="0.6858" z="0.8128">
+        <origin xyz="0 0 0.042916" rpy="0 0 -1.5708"/>
+    </xacro:inertial_box>
     <visual>
       <origin
@@ -140,5 +127,5 @@
         rpy="0 0 0" />
       <mass
-        value="0.37248" />
+        value="0.25" />
       <inertia
         ixx="0.0013774"
@@ -196,5 +183,5 @@
         rpy="0 0 0" />
       <mass
-        value="1.1605" />
+        value="0.1" />
       <inertia
         ixx="0.0053422"
@@ -252,5 +239,5 @@
         rpy="0 0 0" />
       <mass
-        value="1.1605" />
+        value="0.1" />
       <inertia
         ixx="0.0053422"

File: robot_library/src/articubot_one/description/gazebo_control.xacro (robot description, xacro)
@@ -10,5 +10,5 @@
             <!-- Limits -->
             <max_wheel_torque>100</max_wheel_torque>
-            <max_wheel_acceleration>5.0</max_wheel_acceleration>
+            <max_wheel_acceleration>10.0</max_wheel_acceleration>
             <!-- Output -->
             <odometry_frame>odom</odometry_frame>

File: robot_library/src/articubot_one/description/lidar.xacro (robot description, xacro)
@@ -4,5 +4,5 @@
         <parent link="base_link"/>
         <child link="laser_frame"/>
-        <origin xyz="0.122 0 0.4" rpy="0 0 0"/>
+        <origin xyz="-0.30175 0 0.4" rpy="0 0 0"/>
     </joint>
     <link name="laser_frame">
@@ -13,5 +13,5 @@
             <material name="black"/>
         </visual>
-        <visual>
+        <!-- <visual>
             <origin xyz="0 0 -0.05"/>
             <geometry>
@@ -19,5 +19,5 @@
             </geometry>
             <material name="black"/>
-        </visual>
+        </visual> -->
         <collision>
             <geometry>

File: robot_library/src/articubot_one/description/ros2_control.xacro (robot description, xacro)
@@ -15,6 +15,6 @@
             <joint name="left_wheel_joint">
                 <command_interface name="velocity">
-                    <param name="min">-5</param>
-                    <param name="max">5</param>
+                    <param name="min">-2</param>
+                    <param name="max">2</param>
                 </command_interface>
                 <state_interface name="velocity"/>
@@ -23,6 +23,6 @@
             <joint name="right_wheel_joint">
                 <command_interface name="velocity">
-                    <param name="min">-5</param>
-                    <param name="max">5</param>
+                    <param name="min">-2</param>
+                    <param name="max">2</param>
                 </command_interface>
                 <state_interface name="velocity"/>
